Commit message: Updated URDF files and other modifications

File: kuka_description/urdf/depth_camera.xacro (robot description, xacro)
@@ -5,5 +5,5 @@
         <parent link="end_effector_link"/>
         <child link="camera_link"/>
-        <origin xyz="-0.075 0 0" rpy="0 ${PI/2} 0"/>
+        <origin xyz="-0.145 0 0" rpy="0 ${PI/2} 0"/>
     </joint>
     <link name="camera_link">

File: kuka_description/urdf/kuka.urdf.xacro (robot description, xacro)
@@ -215,16 +215,16 @@
         <xacro:default_inertial mass="0.1" />
         <visual>
-            <origin xyz="0.075 0 0.075" rpy="0 0 0" />
-            <geometry>
-                <box size="0.3 0.15 0.15" /> <!-- x, y, z 방향 크기 지정 -->
-            </geometry>
-            <material name="">
-                <color rgba="0 0 0 1"/>
-            </material>
-        </visual>
-        <collision>
-            <origin xyz="0 0 0" rpy="0 0 0" />
-            <geometry>
-                <box size="0.3 0.15 0.15" /> <!-- x, y, z 방향 크기 지정 -->
+            <origin xyz="0.1125 0 0" rpy="0 0 0" />
+            <geometry>
+                <box size="0.3 0.225 0.225" /> <!-- x, y, z 방향 크기 지정 -->
+            </geometry>
+            <material name="">
+                <color rgba="0 0 0 1"/>
+            </material>
+        </visual>
+        <collision>
+            <origin xyz="0.1125 0 0" rpy="0 0 0" />
+            <geometry>
+                <box size="0.3 0.225 0.225" /> <!-- x, y, z 방향 크기 지정 -->
             </geometry>
         </collision>
@@ -233,5 +233,5 @@
         <parent link="link_6" />
         <child link="end_effector_link" />
-        <origin xyz="0.075 0 -0.225" rpy="0 -${PI/2} 0" />
+        <origin xyz="0 0 -0.21" rpy="0 -${PI/2} ${PI/18}" />
         <axis xyz="0 0 1"/>
         <limit lower="0" upper="0"
@@ -241,16 +241,16 @@
         <xacro:default_inertial mass="0.05" />
         <visual>
-            <origin xyz="0 0 0.075" rpy="0 0 0" />
-            <geometry>
-                <cylinder radius="0.01" length="0.15" />
-            </geometry>
-            <material name="">
-                <color rgba="0 0 0 1"/>
-            </material>
-        </visual>
-        <collision>
-            <origin xyz="0 0 0.075" rpy="0 0 0" />
-            <geometry>
-                <cylinder radius="0.01" length="0.15" />
+            <origin xyz="0 0 0.05" rpy="0 0 0" />
+            <geometry>
+                <cylinder radius="0.01" length="0.1" />
+            </geometry>
+            <material name="">
+                <color rgba="0 0 0 1"/>
+            </material>
+        </visual>
+        <collision>
+            <origin xyz="0 0 0.05" rpy="0 0 0" />
+            <geometry>
+                <cylinder radius="0.01" length="0.1" />
             </geometry>
         </collision>
@@ -259,5 +259,5 @@
         <parent link="end_effector_link" />
         <child link="drill_link" />
-        <origin xyz="0 0 -0.15" rpy="0 0 ${PI}" />
+        <origin xyz="0 0 -0.255" rpy="0 0 ${PI}" />
     </joint>
     <transmission name="transmission_end_effector">

File: kuka_description/urdf/realsense_camera.xacro (robot description, xacro)
@@ -4,5 +4,5 @@
     <!-- Joint between the end effector and the D455 camera -->
     <xacro:sensor_d455 parent="end_effector_link" name="camera" use_nominal_extrinsics="true">
-        <origin xyz="-0.075 0 0" rpy="0 ${PI/2} 0" />
+        <origin xyz="-0.145 0 -0.155" rpy="0 ${PI/2} 0" />
     </xacro:sensor_d455>
     <!-- Gazebo 관련 설정 추가 -->
